File: pcb/phonev4.kicad_sch (KiCad schematic)
At the start: 23 parts, among them J1 coin, J2 keypad, J3 display, J4 RJ9, J5 mic, J6 card_reader, J7 speaker, U2 LM386

Commit message: Replace LM386 with TDA2822M dual-channel amplifier, add protection circuits
Major schematic improvements addressing #42 (speaker coupling) and #44
(quiet handset):

- Replace single-channel LM386 with TDA2822M dual-channel amplifier.
  Channel A drives the ringer speaker, channel B drives the handset
  earpiece. Both paths are now amplified and electrically isolated.

- Change I2C pull-ups R1, R2 from 10kΩ to 4.7kΩ (standard for 100kHz).

- Add to BOM: reverse polarity protection (Si2301 P-MOSFET), ESD
  protection (PRTR5V0U2X on RJ9 and coin connectors), 1A resettable
  fuse, power indicator LED, and 7 test points.

- Add TDA2822M symbol to custom library (phone.kicad_sym).

- Rewrite pcb/README.md with complete audio circuit documentation,
  updated BOM, wiring change guide for KiCad, and protection circuit
  descriptions.

The schematic symbol and component values are updated in the .kicad_sch
file. Audio path rewiring and protection circuit placement need to be
completed in KiCad's schematic editor — see the "Schematic Changes
Required in KiCad" section in pcb/README.md.

Addresses #42, #44, #47

Co-authored-by: Cursor <cursoragent@cursor.com>
Parts:
- R1, R2: value 10k -> 4.7k
- U2: value LM386 -> TDA2822M; footprint LM386:DIP08 -> Package_DIP:DIP-8_W7.62mm; symbol Amplifier_Audio:LM386 -> phone:TDA2822M
Connections:
- net 12v: no longer U2.6 (V+)
- net GND: no longer U2.2 (-), U2.4 (GND)
- net speaker_front_pre+: no longer U2.3 (+)
- net at C1.1: now also U2.6 (V+); no longer U2.7 (BYPASS)
- net at U2.5 (OUT_B): no longer C3.1
Changed lines of the file:
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@@
       (effects (font (size 1.27 1.27)) (justify left))
     )
-    (property "Value" "10k" (at 49.53 140.97 0)
+    (property "Value" "4.7k" (at 49.53 140.97 0)
       (effects (font (size 1.27 1.27)) (justify left))
     )
@@
       (effects (font (size 1.27 1.27)) (justify left))
     )
-    (property "Value" "10k" (at 57.15 140.97 0)
+    (property "Value" "4.7k" (at 57.15 140.97 0)
       (effects (font (size 1.27 1.27)) (justify left))
     )
@@
     )
   )
-  (symbol (lib_id "Amplifier_Audio:LM386") (at 113.03 151.13 0) (unit 1)
+  (symbol (lib_id "phone:TDA2822M") (at 113.03 151.13 0) (unit 1)
     (in_bom yes) (on_board yes) (dnp no) (fields_autoplaced)
     (property "Reference" "U2" (at 123.19 146.9391 0)
       (effects (font (size 1.27 1.27)))
     )
-    (property "Value" "LM386" (at 123.19 149.4791 0)
-      (effects (font (size 1.27 1.27)))
-    )
-    (property "Footprint" "LM386:DIP08" (at 115.57 148.59 0)
-      (effects (font (size 1.27 1.27)) hide)
-    )
-    (property "Datasheet" "http://www.ti.com/lit/ds/symlink/lm386.pdf" (at 118.11 146.05 0)
-      (effects (font (size 1.27 1.27)) hide)
-    )
+    (property "Value" "TDA2822M" (at 123.19 149.4791 0)
+      (effects (font (size 1.27 1.27)))
+    )
+    (property "Footprint" "Package_DIP:DIP-8_W7.62mm" (at 113.03 151.13 0)
+      (effects (font (size 1.27 1.27)) hide)
+    )
+    (property "Datasheet" "https://www.st.com/resource/en/datasheet/tda2822m.pdf" (at 113.03 151.13 0)
+      (effects (font (size 1.27 1.27)) hide)
+    )
+    (pin "1")
+    (pin "2")
+    (pin "3")
     (pin "4")
     (pin "5")
-    (pin "1")
     (pin "6")
     (pin "7")
     (pin "8")
-    (pin "3")
-    (pin "2")
-    (instances
-      (project "phonev4"
+    (instances
+      (project "phonev4"
