File: pcb/phonev4.kicad_sch (KiCad schematic)
At the start: 23 parts, among them J1 coin, J2 keypad, J3 display, J4 RJ9, J5 mic, J6 card_reader, J7 speaker, U2 TDA2822M

Commit message: schematic updates
Parts:
- removed C1, C2: CP_Axial_L11.0mm_D8.0mm_P15.00mm, Capacitor_THT:CP_Radial_D8.0mm_P3.80mm, symbol PCM_Capacitor_US_AKL:CP_Axial_L11.0mm_D8.0mm_P15.00mm
- removed C4: 0.1uF_0603_16V, Capacitor_THT:C_Axial_L3.8mm_D2.6mm_P7.50mm_Horizontal, symbol PCM_4ms_Capacitor:0.1uF_0603_16V
- added C_dec, C_inA, C_inB: 100nF, Capacitor_THT:C_Axial_L3.8mm_D2.6mm_P7.50mm_Horizontal, symbol PCM_Capacitor_US_AKL:CP_Axial_L18.0mm_D10.0mm_P25.00mm
- added C_outA, C_vcc: 100µF 16V, Capacitor_THT:CP_Radial_D8.0mm_P2.00mm, symbol PCM_Capacitor_US_AKL:CP_Axial_L18.0mm_D10.0mm_P25.00mm
- added C_ripple: 4.7µF, Capacitor_THT:CP_Radial_D5.0mm_P2.00mm, symbol PCM_Capacitor_US_AKL:CP_Axial_L18.0mm_D10.0mm_P25.00mm
- added D1, D2: PRTR5V0U2X, Package_TO_SOT_SMD:SOT-143, symbol Power_Protection:PRTR5V0U2X
- added D3: Green LED, symbol Device:LED
- added F1: 1A, symbol Device:Fuse
- added Q1: Si2319CDS, Package_TO_SOT_SMD:SOT-23, symbol Transistor_FET:Si2319CDS
- added R3: 1kΩ, Resistor_THT:R_Axial_DIN0204_L3.6mm_D1.6mm_P7.62mm_Horizontal, symbol Device:R_US
- added TP1: 5v, symbol Connector:TestPoint
- added TP2: Pi 3.3v out, symbol Connector:TestPoint
- added TP3: Ground, symbol Connector:TestPoint
- added TP4: SDA, symbol Connector:TestPoint
- added TP5: SCL, symbol Connector:TestPoint
- C_outB: renamed from C3; value CP_Axial_L18.0mm_D10.0mm_P25.00mm -> 100µF 16V; footprint Capacitor_THT:CP_Radial_D10.0mm_P3.80mm -> Capacitor_THT:CP_Radial_D8.0mm_P2.00mm
Connections:
- net 5v: now also C_dec.1, C_vcc.1, D1.4 (VCC), D2.4 (VCC), F1.1, R3.1, TP1.1; no longer U1.1 (IN+)
- net GND: now also U2.2 (GND), C_ripple.2, D1.1 (GND), D2.1 (GND), D3.1 (K), Q1.1 (G), TP3.1
- net coin_rx: now also D2.2 (I/O1)
- net mic+: now also D1.2 (I/O1)
- net scl: now also TP5.1
- net sda: now also TP4.1
- net speaker_front+: now also C_outA.2; no longer C_outB.2
- net speaker_front_pre+: now also C_inA.1
- net speaker_receiver+: now also C_outB.2, D1.3 (I/O2); no longer J7.1 (SIG)
- net at A3.1 (3V3[1]): now also TP2.1
- net at U2.6 (V+): now also C_dec.2, C_vcc.2
- net at U2.1 (OUT_A): now also C_outA.1
- net at U2.3 (IN_A): now also C_inA.2
- net at U2.4 (IN_B): now also C_inB.2
- net at U2.5 (OUT_B): now also C_outB.1
- net at U2.7 (RIPPLE): now also C_ripple.1
- new net: Q1.3 (D), U1.1 (IN+)
- new net: F1.2, Q1.2 (S)
- new net: D3.2 (A), R3.2
- new net speaker_receiver_pre+: C_inB.1, J7.1 (SIG)
Other:
- moved on the sheet: C_outB, U1
