File: pcb/phonev4.kicad_pcb (KiCad board)
At the start: 2 copper layers, 88.9 x 124.5 mm, 25 parts, among them J1 coin, J2 keypad, J3 display, J4 RJ9, J5 mic, J6 card_reader, J7 speaker, U2 LM386

Commit message: PCB: schematic cleanup, cap renames C1-C12, F1 footprint fix, docs
- Rename capacitors to standard refs (C1-C12): C-arduino1->C1, C_inA1->C9, etc.
- F1 footprint: use Capacitor_THT:CP_Radial_D10.0mm_P5.00mm (Fuse_Radial missing in KiCad)
- UNUSED_PINS.md: D2 pin 3 now used (coin_tx)
- SCHEMATIC_LAYOUT.md: layout guide for subsections
- AUDIT.md: wiring verification checked, ERC count 154
- BOM_CHECK.md, phonev4.csv: align with new refs

Co-authored-by: Cursor <cursoragent@cursor.com>
Parts:
- added C10: 100nF, Capacitor_THT:C_Axial_L3.8mm_D2.6mm_P7.50mm_Horizontal, F.Cu at (79.6, 55.1)
- added C11: 100µF 16V, Capacitor_THT:CP_Radial_D8.0mm_P3.80mm, F.Cu at (71.4, 49.5)
- added C6: 100nF, Capacitor_THT:C_Axial_L3.8mm_D2.6mm_P7.50mm_Horizontal, F.Cu at (79.6, 46.8)
- added C7: 100µF 16V, Capacitor_THT:CP_Radial_D8.0mm_P3.80mm, F.Cu at (71.4, 59.0)
- added C8: 4.7µF, Capacitor_THT:CP_Radial_D5.0mm_P2.00mm, F.Cu at (91.0, 72.0)
- added C9: 100nF, Capacitor_THT:C_Axial_L3.8mm_D2.6mm_P7.50mm_Horizontal, F.Cu at (79.6, 51.0)
- added D1: PRTR5V0U2X, Package_TO_SOT_SMD:SOT-143, F.Cu at (70.5, 66.2)
- added D2: PRTR5V0U2X, Package_TO_SOT_SMD:SOT-143, F.Cu at (74.7, 66.2)
- added D3: Green LED, LED_THT:LED_D5.0mm, F.Cu at (70.8, 72.2)
- added F1: 1A, Capacitor_THT:CP_Radial_D10.0mm_P5.00mm, F.Cu at (81.6, 63.0)
- added Q1: Si2319CDS, Package_TO_SOT_SMD:SOT-23, F.Cu at (92.3, 59.4)
- added R3: 1kΩ, Resistor_THT:R_Axial_DIN0204_L3.6mm_D1.6mm_P7.62mm_Horizontal, F.Cu at (79.5, 70.3)
- added TP1: 5V_MAIN, TestPoint:TestPoint_Loop_D2.50mm_Drill1.0mm, F.Cu at (66.0, 47.0)
- added TP2: Pi 3.3v out, TestPoint:TestPoint_Loop_D2.50mm_Drill1.0mm, F.Cu at (66.0, 51.7)
- added TP3: Ground, TestPoint:TestPoint_Loop_D2.50mm_Drill1.0mm, F.Cu at (66.0, 56.4)
- added TP4: SDA, TestPoint:TestPoint_Loop_D2.50mm_Drill1.0mm, F.Cu at (66.0, 61.0)
- added TP5: SCL, TestPoint:TestPoint_Loop_D2.50mm_Drill1.0mm, F.Cu at (66.0, 65.7)
- C12: renamed from C3; value CP_Axial_L18.0mm_D10.0mm_P25.00mm -> 100µF 16V; footprint Capacitor_THT:CP_Radial_D10.0mm_P3.80mm -> Capacitor_THT:CP_Radial_D8.0mm_P3.80mm
- R1, R2: value 10k -> 4.7k
- U2: value LM386 -> TDA2822M; footprint LM386:DIP08 -> Package_DIP:DIP-8_W7.62mm
- renumbered C-arduino1 to C1, C-arduino-display1 to C2, C-card1 to C3, C-coin1 to C4, C-raspi1 to C5
Connections:
- A1 pad GND1: gnd -> GND
- A1 pad GND2: gnd -> GND
- A2 pad GND1: gnd -> GND
- A2 pad GND2: gnd -> GND
- A3 pad 1: unconnected-(A3-3V3[1]-Pad1) -> Net-(A3-3V3[1])
- A3 pad 14: gnd -> GND
- A3 pad 20: gnd -> GND
- A3 pad 25: gnd -> GND
- A3 pad 30: gnd -> GND
- A3 pad 34: gnd -> GND
- A3 pad 39: gnd -> GND
- A3 pad 6: gnd -> GND
- A3 pad 9: gnd -> GND
- C1 pad 2: gnd -> GND
- C12 pad 2: speaker_front+ -> speaker_receiver+
- C2 pad 2: gnd -> GND
- C3 pad 1: gnd -> GND
- C4 pad 2: gnd -> GND
- C5 pad 2: gnd -> GND
- J1 pad 1: gnd -> GND
- J1 pad 4: gnd -> GND
- J1 pad 5: gnd -> GND
- J1 pad 6: gnd -> GND
- J1 pad 7: gnd -> GND
- J1 pad 8: gnd -> GND
- J2 pad 20: gnd -> GND
- J3 pad 26: gnd -> GND
- J4 pad 3: gnd -> GND
- J4 pad 4: gnd -> GND
- J5 pad 2: gnd -> GND
- J6 pad 12: card_seated -> mag_cls
- J6 pad 2: gnd -> GND
- J7 pad 1: speaker_receiver+ -> speaker_receiver_pre+
- J7 pad 2: gnd -> GND
- U1 pad 1: 5V_MAIN -> BOOST_IN+
- U1 pad 2: gnd -> GND
- U1 pad 3: gnd -> GND
- U2 pad 1: unconnected-(U2-GAIN-Pad1) -> Net-(U2-OUT_A)
- U2 pad 2: gnd -> GND
- U2 pad 3: speaker_front_pre+ -> Net-(U2-IN_A)
- U2 pad 4: gnd -> Net-(U2-IN_B)
- U2 pad 6: 12V_COIN -> 5V_MAIN
- U2 pad 7: Net-(U2-BYPASS) -> Net-(U2-RIPPLE)
Routing:
- net 12V_COIN: track 170.7 -> 38.7 mm
- net speaker_front+: track 118.6 -> 0.00 mm
- net gnd: track 111.4 -> 0.00 mm, vias 2 -> 0
- net GND: track 0.00 -> 95.4 mm, vias 0 -> 2
- net speaker_front_pre+: track 48.1 -> 0.00 mm
- net Net-(U2-OUT_B): track 23.7 -> 0.00 mm
- net speaker_receiver+: track 19.6 -> 0.00 mm
- net Net-(U2-BYPASS): track 16.1 -> 0.00 mm
- added copper zone on F.Cu, net GND
- removed copper zone on F.Cu, net gnd
