File: pcb/phonev5.kicad_sch (KiCad schematic)
At the start: 40 parts, among them J1 coin, J2 keypad, J3 display, J4 RJ9, J5 mic, J6 card_reader, J7 speaker, Q1 IRF9540N, U2 TDA2822M

Commit message: Arduino: GPIO reset flashing, remove CMD_FLASH_MODE hack; add CLAUDE.md
Replace the old deploy_display.sh (uhubctl power-cycling, 200-attempt
race loop, CMD_FLASH_MODE silent mode) with a clean GPIO-reset approach
now that the Pi has direct RST connections to both Arduinos:
- GPIO17/GEN0 (pin 11) → Arduino Alpha RST
- GPIO27/GEN2 (pin 13) → Arduino Beta RST (required bodge wire; trace
  missing from phonev5 PCB — documented in pcb/README.md errata)

Changes:
- deploy_display.sh: assert GPIO27 reset (open-drain), wait for device
  to cycle, flash with avrdude; remove uhubctl/1200-baud/race loop
- deploy_keypad.sh: new script, same approach via GPIO17
- Makefile: replace flash_display with deploy_display/deploy_keypad/deploy
- display.ino: remove CMD_FLASH_MODE (0xFF) and silentUntil hack
- pcb/README.md: add Known PCB Errata section for missing Reset 2 trace
- CLAUDE.md: initial project guidance for Claude Code

Co-Authored-By: Claude Sonnet 4.6 <noreply@anthropic.com>
Parts:
- removed C8: 4.7µF, Capacitor_THT:CP_Radial_D5.0mm_P2.00mm, symbol PCM_Capacitor_US_AKL:CP_Axial_L18.0mm_D10.0mm_P25.00mm
- C1, C10, C2, C3, C4, C5, C6, C9: footprint Capacitor_THT:C_Disc_D5.0mm_W2.5mm_P2.50mm -> Capacitor_SMD:C_0805_2012Metric; LCSC C600221 -> C49678
- C11, C12, C7: footprint Capacitor_THT:CP_Radial_D5.0mm_P2.00mm -> Capacitor_SMD:CP_Elec_6.3x5.4; LCSC (none) -> C37308
- D1, D2, D3: footprint Diode_THT:D_DO-201AD_P12.70mm_Horizontal -> Diode_SMD:D_SMB; LCSC (none) -> C78395
- D4: value Green LED -> Red LED; footprint LED_THT:LED_D5.0mm -> LED_SMD:LED_0603_1608Metric; LCSC (none) -> C2286
- F1: footprint footprints:Fuse_Radial_D10.0mm_P5.00mm -> Fuse:Fuse_1812_4532Metric; LCSC (none) -> C2649901
- J7: LCSC (none) -> C2884926
- Q1: value IRF9540N -> AO3401A; footprint footprints:TO-220-3_Vertical_GSD -> Package_TO_SOT_SMD:SOT-23; LCSC (none) -> C15127
- R1, R2: footprint Resistor_THT:R_Axial_DIN0204_L3.6mm_D1.6mm_P7.62mm_Horizontal -> Resistor_SMD:R_0805_2012Metric; LCSC (none) -> C17673
- R3, R4, R5: footprint Resistor_THT:R_Axial_DIN0204_L3.6mm_D1.6mm_P7.62mm_Horizontal -> Resistor_SMD:R_0805_2012Metric; LCSC (none) -> C17513
- U2: value TDA2822M -> PT2308-S; footprint Package_DIP:DIP-8_W7.62mm -> Package_SO:SOIC-8_3.9x4.9mm_P1.27mm; symbol phone:TDA2822M -> phone:PT2308-S; LCSC (none) -> C115492
Connections:
- net 5V_MAIN: now also U2.8 (V+); no longer U2.6 (V+)
- net GND: now also U2.4 (GND), U2.6 (INB-)
- net at C10.2: now also U2.5 (IN_B); no longer U2.4 (IN_B)
- net at C12.1: now also U2.7 (OUT_B); no longer U2.5 (OUT_B)
