File: pcb/phonev5.kicad_sch (KiCad schematic)
At the start: 39 parts, among them J1 coin, J2 keypad, J3 display, J4 RJ9, J5 mic, J6 card_reader, J7 speaker, Q1 AO3401A, U2 PT2308-S

Commit message: updated pcb
Parts:
- removed D1, D2, D3: P6KE6.8CA, Diode_SMD:D_SMB, symbol phone:P6KE6.8CA
- D4: footprint LED_SMD:LED_0603_1608Metric -> LED_SMD:LED_0805_2012Metric; LCSC C2286 -> C2297
