File: pcb/phonev5.kicad_pcb (KiCad board)
At the start: 4 copper layers, 81 x 114 mm, 40 parts, among them J1 coin, J2 keypad, J3 display, J4 RJ9, J5 mic, J6 card_reader, J7 speaker, Q1 AO3401A, U2 PT2308-S

Commit message: updated pcb
Parts:
- removed D1, D2, D3: P6KE6.8CA, Diode_SMD:D_SMB
- C8: footprint Capacitor_SMD:C_0402_1005Metric -> Capacitor_SMD:C_0805_2012Metric
- D4: footprint LED_SMD:LED_0603_1608Metric -> LED_SMD:LED_0805_2012Metric
- moved C3 4.90 mm to (118.5, 55.8)
- moved C4 4.90 mm to (118.5, 44.8)
- moved J1 4.90 mm to (98.8, 46.3)
- moved J6 4.90 mm to (93.9, 57.3)
Routing:
- net speaker_receiver_pre+: track 0.00 -> 48.4 mm, vias 0 -> 1
- net RESET2: track 0.00 -> 30.9 mm
- net key_row_3: track 63.6 -> 44.0 mm
- net key_hook_up: track 53.9 -> 72.0 mm
- net PI_RESET1: track 50.6 -> 34.3 mm, vias 0 -> 1
- net 3.3V: track 105.5 -> 121.2 mm
- net key_col_7: track 62.8 -> 77.4 mm, vias 0 -> 1
- net disp_x6: track 49.0 -> 36.8 mm, vias 1 -> 0
- net key_hook_common: track 61.8 -> 73.4 mm
- net coin_reset: track 46.4 -> 57.9 mm, vias 0 -> 1
- net mag_cls: track 79.3 -> 88.8 mm
- net mic+: track 37.8 -> 28.8 mm
- net mag_rcl: track 39.9 -> 47.5 mm, vias 1 -> 0
- net key_row_1: track 51.5 -> 44.1 mm
- net miso: track 25.4 -> 20.3 mm
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