File: pcb/phonev6.kicad_sch (KiCad schematic)
At the start: 36 parts, among them J1 coin, J2 keypad, J3 display, J4 RJ9, J5 mic, J6 card_reader, J7 speaker, Q1 AO3401A, U2 PT2308-S

Commit message: pcb: remove old v4/v5 designs, make phonev6 canonical
phonev6 (the SMD migration, fabricated and installed) is now the only
design. Promote it from the self-contained pcb/phonev6/ working dir up to
the pcb/ root, where v5 used to live, and delete the old v2/v4/v5 design
files, backups, JLCPCB artifacts, and editor cruft (locks, autosave,
.edit-backup snapshots, empty nested dirs).

Update all references off the deleted v5 files: audit_schematic.py (live),
the PCB README design history + file table, AUDIT/DESIGN_OPTIONS/JLCPCB
docs, and repo-root CLAUDE.md/HARDWARE.md/README.md. The Makefile and
export_jlcpcb.sh were already v6-parameterized. The one-shot migration
scripts (add_no_connect.py, patch*.py) keep their original v4/v5 targets
as applied history.

Co-Authored-By: Claude Opus 4.8 (1M context) <noreply@anthropic.com>
Parts:
- added C13, C14, C15, C17: 22u, Capacitor_SMD:C_0805_2012Metric, symbol Device:C_Small
- added C16, C18, C19, C20: 0.1u, Capacitor_SMD:C_0805_2012Metric, symbol Device:C_Small
- added D10, D11: Yellow LED, LED_SMD:LED_0805_2012Metric, symbol Device:LED
- added D12, D13: Blue LED, LED_SMD:LED_0805_2012Metric, symbol Device:LED
- added D5, D6, D7: P6KE6.8CA, Diode_SMD:D_SMB, symbol phone:P6KE6.8CA
- added D8, D9: Green LED, LED_SMD:LED_0805_2012Metric, symbol Device:LED
- added R10: 330, Resistor_SMD:R_0805_2012Metric, symbol Device:R_US
- added R11: 3.3k, Resistor_SMD:R_0805_2012Metric, symbol Device:R_US
- added R12, R13, R14, R15: 1k, Resistor_SMD:R_0805_2012Metric, symbol Device:R_US
- added R6, R7: 10k, Resistor_SMD:R_0805_2012Metric, symbol Device:R_US
- added R8, R9: 4.7, Resistor_SMD:R_0805_2012Metric, symbol Device:R_US
- F1: value 1A -> 2A
- U2: value PT2308-S -> TDA2822M; symbol phone:PT2308-S -> phone:TDA2822M; LCSC C115492 -> C725341
Connections:
- net 12V_COIN: now also C17.1, C18.1, R11.1
- net 3.3V: now also R10.1; no longer A1.3V3 (3.3V), A2.3V3 (3.3V)
- net 5V_MAIN: now also U2.2 (Vcc), D5.1, R12.1, R13.1, R14.1, R15.1; no longer U2.8 (V+)
- net BOOST_IN+: now also C15.1, C16.1
- net GND: now also C13.2, C14.2, C15.2, C16.2, C17.2, C18.2, C19.2, C20.2, D5.2, D6.2, D7.2, D8.1 (K), D9.1 (K), R6.2, R7.2; no longer U2.2 (INA-), U2.6 (INB-)
- net RESET1: now also D10.1 (K)
- net RESET2: now also D11.1 (K)
- net scl: now also D13.1 (K)
- net sda: now also D12.1 (K)
- net speaker_front+: now also D6.1, R8.1
- net speaker_receiver+: now also D7.1, R9.1
- net at U2.3 (OUT2): now also C12.1; no longer C9.2
- net AMP_IN2: now reaches C10.2
- net AMP_IN2: now also U2.6 (IN2), R7.1; no longer U2.5 (IN_B)
- net AMP_IN1: now reaches U2.7 (IN1)
- net AMP_IN1: now also C9.2, R6.1; no longer C12.1
- new net LED_12V: D9.2 (A), R11.2
- new net LED_3V3: D8.2 (A), R10.2
- new net LED_RST1: D10.2 (A), R12.2
- new net LED_RST2: D11.2 (A), R13.2
- new net LED_SCL: D13.2 (A), R15.2
- new net LED_SDA: D12.2 (A), R14.2
- new net NF1: C13.1, U2.8 (NF1)
- new net NF2: C14.1, U2.5 (NF2)
- new net ZOBEL1: C19.1, R8.2
- new net ZOBEL2: C20.1, R9.2
- no-connect marks 55 -> 57
